Commit message: Added new meshes to prevent collision error in the scenario
The error is that the meshes have not manifold faces.

File: kuka_kr210_support/urdf/kr210r3100_macro.xacro (robot description, xacro)
@@ -22,5 +22,5 @@
         <origin rpy="0 0 0" xyz="0 0 0"/>
         <geometry>
-          <mesh filename="file://$(find kuka_kr210_support)/meshes/kr210r3100/collision/base_link.stl" scale="0.001 0.001 0.001"/>
+          <mesh filename="file://$(find maurob_gripper_description)/meshes/kr210r3100/collision/base_link2.stl" scale="0.001 0.001 0.001"/>
         </geometry>
       </collision>
@@ -44,5 +44,5 @@
       <origin rpy="0 0 0" xyz="0.0 0.0 0.0"/>
       <geometry>
-        <mesh filename="file://$(find kuka_kr210_support)/meshes/kr210r3100/collision/l1_1.stl" scale="0.001 0.001 0.001"/>
+        <mesh filename="file://$(find kuka_kr210_support)/meshes/kr210r3100/collision/l1_2.stl" scale="0.001 0.001 0.001"/>
       </geometry>
     </collision>

Commit message: Added new meshes to avoid collision error

File: kuka_kr210_support/urdf/kr210r3100_macro.xacro (robot description, xacro)
@@ -22,5 +22,5 @@
         <origin rpy="0 0 0" xyz="0 0 0"/>
         <geometry>
-          <mesh filename="file://$(find maurob_gripper_description)/meshes/kr210r3100/collision/base_link2.stl" scale="0.001 0.001 0.001"/>
+          <mesh filename="file://$(find kuka_kr210_support)/meshes/kr210r3100/collision/base_link.stl" scale="0.001 0.001 0.001"/>
         </geometry>
       </collision>
@@ -44,5 +44,5 @@
       <origin rpy="0 0 0" xyz="0.0 0.0 0.0"/>
       <geometry>
-        <mesh filename="file://$(find kuka_kr210_support)/meshes/kr210r3100/collision/l1_2.stl" scale="0.001 0.001 0.001"/>
+        <mesh filename="file://$(find kuka_kr210_support)/meshes/kr210r3100/collision/l1_1.stl" scale="0.001 0.001 0.001"/>
       </geometry>
     </collision>

Commit message: H-KA KR210

File: kuka_kr210_support/urdf/kr210r3100_macro.xacro (robot description, xacro)
@@ -211,5 +211,5 @@
       <link name="${prefix}base"/>
       <joint name="${prefix}base_link-base" type="fixed">
-          <origin xyz="0 0 0" rpy="0 0 0"/>
+          <origin xyz="0 0 -0.23" rpy="0 0 0"/>
           <parent link="${prefix}base_link"/>
           <child link="${prefix}base"/>
