Commit message: Make kuka hardware async by default

File: kuka_ros2_control_support/urdf/common_kuka.xacro (robot description, xacro)
@@ -3,4 +3,5 @@
   <xacro:arg name="robot_name" default="kuka" />
   <xacro:arg name="prefix" default="" />
+  <xacro:arg name="is_async" default="true" />
   <xacro:arg name="description_package" default="" />
   <xacro:arg name="description_macro_file" default="" />

File: kuka_ros2_control_support/urdf/common_macro.ros2_control.xacro (robot description, xacro)
@@ -21,7 +21,4 @@
       <xacro:property name="is_async" value="false" />
     </xacro:if>
-    <xacro:unless value="${use_mock_hardware}">
-      <xacro:property name="be_async" value="${is_async}" />
-    </xacro:unless>
     <ros2_control name="${name}" type="system" is_async="${is_async}">
       <hardware>

Commit message: Use FZI RSI driver.

File: kuka_ros2_control_support/urdf/common_kuka.xacro (robot description, xacro)
@@ -14,5 +14,4 @@
   <!-- ros2_control mock and simulation plugins -->
   <xacro:arg name="use_mock_hardware" default="false" />
-  <xacro:arg name="use_external_gripper_driver" default="true" />
   <xacro:arg name="sim_gazebo_classic" default="false" />
   <xacro:arg name="sim_gazebo" default="false" />
@@ -26,4 +25,5 @@
   <xacro:include filename="$(find ${description_package})/urdf/${description_macro_file}"/>
   <xacro:include filename="$(find kuka_ros2_control_support)/urdf/common_macro.ros2_control.xacro"/>
+  <!-- add ros2_control KUKA plugin -->
   <xacro:kuka_common_ros2_control_macro
     name="$(arg robot_name)"
@@ -43,4 +43,5 @@
     initial_positions="${xacro.load_yaml(initial_positions_file)}"
   />
+  <!-- load description accorind to the package and macro name -->
   <xacro:if value="${description_package == 'kuka_kr3_support'}">
     <xacro:kuka_kr3r540 prefix="$(arg prefix)"/>

File: kuka_ros2_control_support/urdf/common_macro.ros2_control.xacro (robot description, xacro)
@@ -1,8 +1,18 @@
 <?xml version="1.0"?>
 <robot xmlns:xacro="http://www.ros.org/wiki/xacro">
+  <xacro:macro name="kuka_rsi_driver_control_joint" params="name initial_position">
+    <joint name="${name}">
+      <command_interface name="position" />
+      <state_interface name="position">
+        <param name="initial_value">${initial_position}</param>
+      </state_interface>
+      <state_interface name="effort" />
+    </joint>
+  </xacro:macro>
   <xacro:macro name="kuka_common_ros2_control_macro" params="
                name
                prefix
                is_async:=^|true
+               rw_rate:=^|250
                use_eki_communication:=^|false
                eki_robot_ip:=^|127.0.0.1
@@ -12,5 +22,6 @@
                rsi_listen_port:=^|49152
                use_mock_hardware:=^|false
-               sim_gazebo_classic:=^|false
+               mock_gpio_commands:=^|false
+               mock_sensor_commands:=^|false
                sim_gazebo:=^|false
                simulation_controllers
@@ -18,17 +29,16 @@
                initial_positions:=${dict(joint_a1=0.0,joint_a2=-1.57,joint_a3=1.57,joint_a4=0.0,joint_a5=1.57,joint_a6=0.0)}"
                >
-    <xacro:if value="${use_mock_hardware}">
+    <xacro:if value="$(eval ${use_mock_hardware} or ${sim_gazebo})">
       <xacro:property name="is_async" value="false" />
     </xacro:if>
-    <ros2_control name="${name}" type="system" is_async="${is_async}">
+    <ros2_control name="${name}" type="system" is_async="${is_async}" rw_rate="${rw_rate}">
       <hardware>
         <xacro:if value="${use_mock_hardware}">
           <plugin>mock_components/GenericSystem</plugin>
-        </xacro:if>
-        <xacro:if value="${sim_gazebo_classic}">
-          <plugin>gazebo_ros2_control/GazeboSystem</plugin>
+          <param name="mock_gpio_commands">${mock_gpio_commands}</param>
+          <param name="mock_sensor_commands">${mock_sensor_commands}</param>
         </xacro:if>
         <xacro:if value="${sim_gazebo}">
-          <plugin>ign_ros2_control/IgnitionSystem</plugin>
+          <plugin>gz_ros2_control/GzSystem</plugin>
         </xacro:if>
         <xacro:if value="${use_eki_communication}">
@@ -38,91 +48,58 @@
         </xacro:if>
         <xacro:if value="${use_rsi_communication}">
-          <plugin>kuka_rsi_hw_interface/RobotControlInterface</plugin>
+          <plugin>kuka_rsi_driver/KukaRsiHardwareInterface</plugin>
           <param name="listen_address">${rsi_listen_ip}</param>
           <param name="listen_port">${rsi_listen_port}</param>
         </xacro:if>
       </hardware>
-      <joint name="${prefix}joint_a1">
-        <command_interface name="position">
-          <param name="min">-1</param>
-          <param name="max">1</param>
-        </command_interface>
-        <state_interface name="position">
-          <param name="initial_value">${initial_positions['joint_a1']}</param>
+      <xacro:kuka_rsi_driver_control_joint name="${prefix}joint_a1" initial_position="${initial_positions['joint_a1']}" />
+      <xacro:kuka_rsi_driver_control_joint name="${prefix}joint_a2" initial_position="${initial_positions['joint_a2']}" />
+      <xacro:kuka_rsi_driver_control_joint name="${prefix}joint_a3" initial_position="${initial_positions['joint_a3']}" />
+      <xacro:kuka_rsi_driver_control_joint name="${prefix}joint_a4" initial_position="${initial_positions['joint_a4']}" />
+      <xacro:kuka_rsi_driver_control_joint name="${prefix}joint_a5" initial_position="${initial_positions['joint_a5']}" />
+      <xacro:kuka_rsi_driver_control_joint name="${prefix}joint_a6" initial_position="${initial_positions['joint_a6']}" />
+      <xacro:if value="${description_package == 'kuka_lbr_iiwa_support'}">
+        <xacro:kuka_rsi_driver_control_joint name="${prefix}joint_a7" initial_position="${initial_positions['joint_a7']}" />
+      </xacro:if>
+      <sensor name="${prefix}tcp">
+        <state_interface name="position.x">
+          <param name="initial_value">0</param>
         </state_interface>
-      </joint>
-      <joint name="${prefix}joint_a2">
-        <command_interface name="position">
-          <param name="min">-1</param>
-          <param name="max">1</param>
-        </command_interface>
-        <state_interface name="position">
-          <param name="initial_value">${initial_positions['joint_a2']}</param>
+        <state_interface name="position.y">
+          <param name="initial_value">0</param>
         </state_interface>
-	  </joint>
-      <joint name="${prefix}joint_a3">
-        <command_interface name="position">
-          <param name="min">-1</param>
-          <param name="max">0.61</param>
-        </command_interface>
-        <state_interface name="position">
-          <param name="initial_value">${initial_positions['joint_a3']}</param>
+        <state_interface name="position.z">
+          <param name="initial_value">0</param>
         </state_interface>
-	  </joint>
-      <joint name="${prefix}joint_a4">
-        <command_interface name="position">
-          <param name="min">-1</param>
-          <param name="max">1</param>
-        </command_interface>
-        <state_interface name="position">
-          <param name="initial_value">${initial_positions['joint_a4']}</param>
+        <state_interface name="orientation.x">
+          <param name="initial_value">0</param>
         </state_interface>
-      </joint>
-      <joint name="${prefix}joint_a5">
-        <command_interface name="position">
-          <param name="min">-1</param>
-          <param name="max">1</param>
-        </command_interface>
-        <state_interface name="position">
-          <param name="initial_value">${initial_positions['joint_a5']}</param>
+        <state_interface name="orientation.y">
+          <param name="initial_value">0</param>
         </state_interface>
-      </joint>
-      <joint name="${prefix}joint_a6">
-        <command_interface name="position">
-          <param name="min">-1</param>
-          <param name="max">1</param>
-        </command_interface>
-        <state_interface name="position">
-          <param name="initial_value">${initial_positions['joint_a6']}</param>
+        <state_interface name="orientation.z">
+          <param name="initial_value">0</param>
         </state_interface>
-      </joint>
-      <xacro:if value="${description_package == 'kuka_lbr_iiwa_support'}">
-        <joint name="${prefix}joint_a7">
-        <command_interface name="position">
-          <param name="min">-1</param>
-          <param name="max">1</param>
-        </command_interface>
-        <state_interface name="position">
-          <param name="initial_value">${initial_positions['joint_a7']}</param>
+        <state_interface name="orientation.w">
+          <param name="initial_value">1</param>
         </state_interface>
-        </joint>
-      </xacro:if>
+      </sensor>
+      <gpio name="${prefix}robot_state">
+        <state_interface name="program_state">
+          <param name="initial_value">3</param>
+        </state_interface>
+      </gpio>
+      <gpio name="${prefix}speed_scaling">
+        <state_interface name="speed_scaling_factor">
+          <param name="initial_value">1</param>
+        </state_interface>
+      </gpio>
     </ros2_control>
-    <xacro:if value="$(arg sim_gazebo_classic)">
+    <xacro:if value="${sim_gazebo}">
       <!-- Gazebo plugins -->
       <gazebo reference="world">
       </gazebo>
       <gazebo>
-        <plugin filename="libgazebo_ros2_control.so" name="gazebo_ros2_control">
-          <parameters>${simulation_controllers}</parameters>
-        </plugin>
-      </gazebo>
-    </xacro:if>
-    <xacro:if value="$(arg sim_gazebo)">
-      <!-- Gazebo plugins -->
-      <gazebo reference="world">
-      </gazebo>
-      <gazebo>
-        <plugin filename="libign_ros2_control-system.so" name="ign_ros2_control::IgnitionROS2ControlPlugin">
+        <plugin filename="libgz_ros2_control-system.so" name="gz_ros2_control::GzROS2ControlPlugin">
           <parameters>${simulation_controllers}</parameters>
           <controller_manager_node_name>${prefix}controller_manager</controller_manager_node_name>
