Commit message: Don't start as async is MockHW.

File: kuka_ros2_control_support/urdf/common_macro.ros2_control.xacro (robot description, xacro)
@@ -18,4 +18,10 @@
                initial_positions:=${dict(joint_a1=0.0,joint_a2=-1.57,joint_a3=1.57,joint_a4=0.0,joint_a5=1.57,joint_a6=0.0)}"
                >
+    <xacro:if value="${use_mock_hardware}">
+      <xacro:property name="is_async" value="false" />
+    </xacro:if>
+    <xacro:unless value="${use_mock_hardware}">
+      <xacro:property name="be_async" value="${is_async}" />
+    </xacro:unless>
     <ros2_control name="${name}" type="system" is_async="${is_async}">
       <hardware>

Commit message: added  use_motion_primitives_driver parameter -->  use MotionPrimitivesKukaDriver, use joints without command interfaces and add "gpio" motion_primitive

File: kuka_ros2_control_support/urdf/common_macro.ros2_control.xacro (robot description, xacro)
@@ -6,4 +6,5 @@
                is_async:=^|true
                use_eki_communication:=^|false
+               use_motion_primitives_driver:=^|false
                eki_robot_ip:=^|127.0.0.1
                eki_robot_port:=^|54600
@@ -40,4 +41,9 @@
           <param name="eki_robot_port">${eki_robot_port}</param>
         </xacro:if>
+        <xacro:if value="${use_motion_primitives_driver}">
+          <plugin>kuka_eki_motion_primitives_hw_interface/MotionPrimitivesKukaDriver</plugin>
+          <param name="robot_ip">${eki_robot_ip}</param>
+          <param name="eki_robot_port">${eki_robot_port}</param>
+        </xacro:if>
         <xacro:if value="${use_rsi_communication}">
           <plugin>kuka_rsi_hw_interface/RobotControlInterface</plugin>
@@ -46,58 +52,126 @@
         </xacro:if>
       </hardware>
-      <joint name="${prefix}joint_a1">
-        <command_interface name="position">
-          <param name="min">-1</param>
-          <param name="max">1</param>
-        </command_interface>
-        <state_interface name="position">
-          <param name="initial_value">${initial_positions['joint_a1']}</param>
-        </state_interface>
-      </joint>
-      <joint name="${prefix}joint_a2">
-        <command_interface name="position">
-          <param name="min">-1</param>
-          <param name="max">1</param>
-        </command_interface>
-        <state_interface name="position">
-          <param name="initial_value">${initial_positions['joint_a2']}</param>
-        </state_interface>
-	  </joint>
-      <joint name="${prefix}joint_a3">
-        <command_interface name="position">
-          <param name="min">-1</param>
-          <param name="max">0.61</param>
-        </command_interface>
-        <state_interface name="position">
-          <param name="initial_value">${initial_positions['joint_a3']}</param>
-        </state_interface>
-	  </joint>
-      <joint name="${prefix}joint_a4">
-        <command_interface name="position">
-          <param name="min">-1</param>
-          <param name="max">1</param>
-        </command_interface>
-        <state_interface name="position">
-          <param name="initial_value">${initial_positions['joint_a4']}</param>
-        </state_interface>
-      </joint>
-      <joint name="${prefix}joint_a5">
-        <command_interface name="position">
-          <param name="min">-1</param>
-          <param name="max">1</param>
-        </command_interface>
-        <state_interface name="position">
-          <param name="initial_value">${initial_positions['joint_a5']}</param>
-        </state_interface>
-      </joint>
-      <joint name="${prefix}joint_a6">
-        <command_interface name="position">
-          <param name="min">-1</param>
-          <param name="max">1</param>
-        </command_interface>
-        <state_interface name="position">
-          <param name="initial_value">${initial_positions['joint_a6']}</param>
-        </state_interface>
-      </joint>
+      <!-- Dont use command interfaces for joints if use_motion_primitives_driver is true-->
+      <xacro:if value="${use_motion_primitives_driver}">
+        <joint name="${prefix}joint_a1">
+          <state_interface name="position">
+            <param name="initial_value">${initial_positions['joint_a1']}</param>
+          </state_interface>
+        </joint>
+        <joint name="${prefix}joint_a2">
+          <state_interface name="position">
+            <param name="initial_value">${initial_positions['joint_a2']}</param>
+          </state_interface>
+      </joint>
+        <joint name="${prefix}joint_a3">
+          <state_interface name="position">
+            <param name="initial_value">${initial_positions['joint_a3']}</param>
+          </state_interface>
+      </joint>
+        <joint name="${prefix}joint_a4">
+          <state_interface name="position">
+            <param name="initial_value">${initial_positions['joint_a4']}</param>
+          </state_interface>
+        </joint>
+        <joint name="${prefix}joint_a5">
+          <state_interface name="position">
+            <param name="initial_value">${initial_positions['joint_a5']}</param>
+          </state_interface>
+        </joint>
+        <joint name="${prefix}joint_a6">
+          <state_interface name="position">
+            <param name="initial_value">${initial_positions['joint_a6']}</param>
+          </state_interface>
+        </joint>
+      </xacro:if>
+      <!-- Use command interfaces for joints if use_motion_primitives_driver is false-->
+      <xacro:unless value="${use_motion_primitives_driver}">
+        <joint name="${prefix}joint_a1">
+          <command_interface name="position">
+            <param name="min">-1</param>
+            <param name="max">1</param>
+          </command_interface>
+          <state_interface name="position">
+            <param name="initial_value">${initial_positions['joint_a1']}</param>
+          </state_interface>
+        </joint>
+        <joint name="${prefix}joint_a2">
+          <command_interface name="position">
+            <param name="min">-1</param>
+            <param name="max">1</param>
+          </command_interface>
+          <state_interface name="position">
+            <param name="initial_value">${initial_positions['joint_a2']}</param>
+          </state_interface>
+      </joint>
+        <joint name="${prefix}joint_a3">
+          <command_interface name="position">
+            <param name="min">-1</param>
+            <param name="max">0.61</param>
+          </command_interface>
+          <state_interface name="position">
+            <param name="initial_value">${initial_positions['joint_a3']}</param>
+          </state_interface>
+      </joint>
+        <joint name="${prefix}joint_a4">
+          <command_interface name="position">
+            <param name="min">-1</param>
+            <param name="max">1</param>
+          </command_interface>
+          <state_interface name="position">
+            <param name="initial_value">${initial_positions['joint_a4']}</param>
+          </state_interface>
+        </joint>
+        <joint name="${prefix}joint_a5">
+          <command_interface name="position">
+            <param name="min">-1</param>
+            <param name="max">1</param>
+          </command_interface>
+          <state_interface name="position">
+            <param name="initial_value">${initial_positions['joint_a5']}</param>
+          </state_interface>
+        </joint>
+        <joint name="${prefix}joint_a6">
+          <command_interface name="position">
+            <param name="min">-1</param>
+            <param name="max">1</param>
+          </command_interface>
+          <state_interface name="position">
+            <param name="initial_value">${initial_positions['joint_a6']}</param>
+          </state_interface>
+        </joint>
+      </xacro:unless>
+      <!-- Interfaces for motion_primitives_driver if  use_motion_primitives_driver==true-->
+      <xacro:if value="${use_motion_primitives_driver}">
+        <gpio name="motion_primitive">
+          <command_interface name="motion_type"/>
+          <command_interface name="q1"/>
+          <command_interface name="q2"/>
+          <command_interface name="q3"/>
+          <command_interface name="q4"/>
+          <command_interface name="q5"/>
+          <command_interface name="q6"/>
+          <command_interface name="pos_x"/>
+          <command_interface name="pos_y"/>
+          <command_interface name="pos_z"/>
+          <command_interface name="pos_qx"/>
+          <command_interface name="pos_qy"/>
+          <command_interface name="pos_qz"/>
+          <command_interface name="pos_qw"/>
+          <command_interface name="pos_via_x"/>
+          <command_interface name="pos_via_y"/>
+          <command_interface name="pos_via_z"/>
+          <command_interface name="pos_via_qx"/>
+          <command_interface name="pos_via_qy"/>
+          <command_interface name="pos_via_qz"/>
+          <command_interface name="pos_via_qw"/>
+          <command_interface name="blend_radius"/>
+          <command_interface name="velocity"/>
+          <command_interface name="acceleration"/>
+          <command_interface name="move_time"/>
+          <state_interface name="execution_status"/>
+          <state_interface name="ready_for_new_primitive"/>
+        </gpio>
+      </xacro:if>
       <xacro:if value="${description_package == 'kuka_lbr_iiwa_support'}">
         <joint name="${prefix}joint_a7">

Commit message: fixed formatting (only white spaces)

File: kuka_ros2_control_support/urdf/common_macro.ros2_control.xacro (robot description, xacro)
@@ -63,14 +63,14 @@
             <param name="initial_value">${initial_positions['joint_a2']}</param>
           </state_interface>
-      </joint>
-        <joint name="${prefix}joint_a3">
-          <state_interface name="position">
-            <param name="initial_value">${initial_positions['joint_a3']}</param>
-          </state_interface>
-      </joint>
-        <joint name="${prefix}joint_a4">
-          <state_interface name="position">
-            <param name="initial_value">${initial_positions['joint_a4']}</param>
-          </state_interface>
+        </joint>
+          <joint name="${prefix}joint_a3">
+            <state_interface name="position">
+              <param name="initial_value">${initial_positions['joint_a3']}</param>
+            </state_interface>
+        </joint>
+          <joint name="${prefix}joint_a4">
+            <state_interface name="position">
+              <param name="initial_value">${initial_positions['joint_a4']}</param>
+            </state_interface>
         </joint>
         <joint name="${prefix}joint_a5">
@@ -104,5 +104,5 @@
             <param name="initial_value">${initial_positions['joint_a2']}</param>
           </state_interface>
-      </joint>
+        </joint>
         <joint name="${prefix}joint_a3">
           <command_interface name="position">
@@ -113,5 +113,5 @@
             <param name="initial_value">${initial_positions['joint_a3']}</param>
           </state_interface>
-      </joint>
+        </joint>
         <joint name="${prefix}joint_a4">
           <command_interface name="position">

Commit message: Make ros2_control common file EKI compatible.

File: kuka_ros2_control_support/urdf/common_macro.ros2_control.xacro (robot description, xacro)
@@ -1,5 +1,5 @@
 <?xml version="1.0"?>
 <robot xmlns:xacro="http://www.ros.org/wiki/xacro">
-  <xacro:macro name="kuka_rsi_driver_control_joint" params="name initial_position">
+  <xacro:macro name="kuka_rsi_driver_control_joint" params="name initial_position use_eki_communication:=^|false">
     <joint name="${name}">
       <command_interface name="position" />
@@ -7,5 +7,7 @@
         <param name="initial_value">${initial_position}</param>
       </state_interface>
-      <state_interface name="effort" />
+      <xacro:unless value="${use_eki_communication}">
+        <state_interface name="effort" />
+      </xacro:unless>
     </joint>
   </xacro:macro>
@@ -62,37 +64,39 @@
         <xacro:kuka_rsi_driver_control_joint name="${prefix}joint_a7" initial_position="${initial_positions['joint_a7']}" />
       </xacro:if>
-      <sensor name="${prefix}tcp">
-        <state_interface name="position.x">
-          <param name="initial_value">0</param>
-        </state_interface>
-        <state_interface name="position.y">
-          <param name="initial_value">0</param>
-        </state_interface>
-        <state_interface name="position.z">
-          <param name="initial_value">0</param>
-        </state_interface>
-        <state_interface name="orientation.x">
-          <param name="initial_value">0</param>
-        </state_interface>
-        <state_interface name="orientation.y">
-          <param name="initial_value">0</param>
-        </state_interface>
-        <state_interface name="orientation.z">
-          <param name="initial_value">0</param>
-        </state_interface>
-        <state_interface name="orientation.w">
-          <param name="initial_value">1</param>
-        </state_interface>
-      </sensor>
-      <gpio name="${prefix}robot_state">
-        <state_interface name="program_state">
-          <param name="initial_value">3</param>
-        </state_interface>
-      </gpio>
-      <gpio name="${prefix}speed_scaling">
-        <state_interface name="speed_scaling_factor">
-          <param name="initial_value">1</param>
-        </state_interface>
-      </gpio>
+      <xacro:unless value="${use_eki_communication}">
+        <sensor name="${prefix}tcp">
+          <state_interface name="position.x">
+            <param name="initial_value">0</param>
+          </state_interface>
+          <state_interface name="position.y">
+            <param name="initial_value">0</param>
+          </state_interface>
+          <state_interface name="position.z">
+            <param name="initial_value">0</param>
+          </state_interface>
+          <state_interface name="orientation.x">
+            <param name="initial_value">0</param>
+          </state_interface>
+          <state_interface name="orientation.y">
+            <param name="initial_value">0</param>
+          </state_interface>
+          <state_interface name="orientation.z">
+            <param name="initial_value">0</param>
+          </state_interface>
+          <state_interface name="orientation.w">
+            <param name="initial_value">1</param>
+          </state_interface>
+        </sensor>
+        <gpio name="${prefix}robot_state">
+          <state_interface name="program_state">
+            <param name="initial_value">3</param>
+          </state_interface>
+        </gpio>
+        <gpio name="${prefix}speed_scaling">
+          <state_interface name="speed_scaling_factor">
+            <param name="initial_value">1</param>
+          </state_interface>
+        </gpio>
+      </xacro:unless>
     </ros2_control>
     <xacro:if value="${sim_gazebo}">

Commit message: EKI Configuration working.

File: kuka_ros2_control_support/urdf/common_macro.ros2_control.xacro (robot description, xacro)
@@ -31,4 +31,8 @@
                initial_positions:=${dict(joint_a1=0.0,joint_a2=-1.57,joint_a3=1.57,joint_a4=0.0,joint_a5=1.57,joint_a6=0.0)}"
                >
+    <xacro:if value="${use_eki_communication}">
+      <xacro:property name="is_async" value="true" />
+      <xacro:property name="rw_rate" value="75" />
+    </xacro:if>
     <xacro:if value="$(eval ${use_mock_hardware} or ${sim_gazebo})">
       <xacro:property name="is_async" value="false" />
